Commit message: [wr8_soft] Fixed TF system position

File: wr8_description/urdf/model.urdf.xacro (robot description, xacro)
@@ -169,5 +169,5 @@
     <child link="base_link"/>
     <!-- <origin xyz="${wheelbase/2} 0 ${wheel_radius}" rpy="0 0 0"/> -->
-    <origin xyz="0 0 ${wheel_radius}" rpy="0 0 0"/>
+    <origin xyz="${wheelbase/2} 0 ${wheel_radius}" rpy="0 0 0"/>
   </joint>
 <!--

Commit message: [wr8_soft] Multiple fixes for graph path integration

File: wr8_description/urdf/model.urdf.xacro (robot description, xacro)
@@ -163,5 +163,9 @@
   </link>
   <gazebo reference="base_link">
-    <material>Gazebo/Grey</material>
+    <!-- <visual>   -->
+      <material>
+        Gazebo/Orange
+      </material>
+    <!-- </visual> -->
   </gazebo>
   <joint name="base_footage_2_link" type="fixed">

Commit message: [ROS] fixed collisions with base_* frames - only base_link left

File: wr8_description/urdf/model.urdf.xacro (robot description, xacro)
@@ -140,8 +140,12 @@
     </transmission> -->
   </xacro:macro>
+  <!-- base_footprint - base_link on floor -->
   <link name="base_footprint">
   </link>
   <gazebo reference="base_footprint"/>
   <link name="base_link">
+  </link>
+  <gazebo reference="base_link"/>
+  <link name="base_center">
     <visual>
       <origin xyz="0 0 0" rpy="0 0 0" />
@@ -162,5 +166,5 @@
     </xacro:solid_cuboid_inertial>
   </link>
-  <gazebo reference="base_link">
+  <gazebo reference="base_center">
     <!-- <visual>   -->
       <material>
@@ -172,16 +176,21 @@
     <parent link="base_footprint"/>
     <child link="base_link"/>
-    <!-- <origin xyz="${wheelbase/2} 0 ${wheel_radius}" rpy="0 0 0"/> -->
+    <!-- base_footprint - base_link on floor -->
+    <origin xyz="0 0 ${wheel_radius}" rpy="0 0 0"/>
+  </joint>
+  <joint name="base_footage_2_center" type="fixed">
+    <parent link="base_footprint"/>
+    <child link="base_center"/>
     <origin xyz="${wheelbase/2} 0 ${wheel_radius}" rpy="0 0 0"/>
   </joint>
 <!--
-  <xacro:steering_wheel name="right_steer_wheel" base_name="base_link" xyz="${wheelbase/2} ${-chassis_width/2} 0" ref="-1" />
-  <xacro:steering_wheel name="left_steer_wheel" base_name="base_link" xyz="${wheelbase/2} ${chassis_width/2} 0" ref="1" />
+  <xacro:steering_wheel name="right_steer_wheel" base_name="base_center" xyz="${wheelbase/2} ${-chassis_width/2} 0" ref="-1" />
+  <xacro:steering_wheel name="left_steer_wheel" base_name="base_center" xyz="${wheelbase/2} ${chassis_width/2} 0" ref="1" />
  -->
-  <xacro:steering_wheel name="right_steer_wheel" base_name="base_link" xyz="${wheelbase/2} ${-(chassis_width/2 + wheel_chassis_bias)} ${-chassis_height/2}" ref="-1" />
-  <xacro:steering_wheel name="left_steer_wheel" base_name="base_link" xyz="${wheelbase/2} ${(chassis_width/2 + wheel_chassis_bias)} ${-chassis_height/2}" ref="1" />
-  <xacro:traveling_wheel name="right_travel_wheel" base_name="base_link"
+  <xacro:steering_wheel name="right_steer_wheel" base_name="base_center" xyz="${wheelbase/2} ${-(chassis_width/2 + wheel_chassis_bias)} ${-chassis_height/2}" ref="-1" />
+  <xacro:steering_wheel name="left_steer_wheel" base_name="base_center" xyz="${wheelbase/2} ${(chassis_width/2 + wheel_chassis_bias)} ${-chassis_height/2}" ref="1" />
+  <xacro:traveling_wheel name="right_travel_wheel" base_name="base_center"
                          xyz="${-wheelbase/2} ${-(chassis_width/2 + wheel_chassis_bias)} ${-chassis_height/2}" />
-  <xacro:traveling_wheel name="left_travel_wheel" base_name="base_link"
+  <xacro:traveling_wheel name="left_travel_wheel" base_name="base_center"
                          xyz="${-wheelbase/2} ${(chassis_width/2 + wheel_chassis_bias)} ${-chassis_height/2}" />
   <!-- Gazebo plugin for ROS Control -->
@@ -191,7 +200,8 @@
     </plugin>
   </gazebo>
+  <!-- Setup LIDAR -->
   <xacro:property name="lidar_height" value="0.04"/>
   <xacro:property name="lidar_radius" value="0.04"/>
-  <link name="hokuyo_link">
+  <link name="laser_frame">
     <xacro:solid_cylinder_inertial
         r="${lidar_radius}" h="${lidar_height}"
@@ -213,9 +223,10 @@
   </link>
   <joint name="hokuyo_joint" type="fixed">
-    <child link="hokuyo_link" />
+    <child link="laser_frame" />
     <parent link="base_link" />
-    <origin xyz="0 0 ${chassis_height/2 + lidar_height/2}" />
+    <!-- Taken from physical parameters (wr8_software/launch/base/lidar.launch) -->
+    <origin xyz="0.14 0 0.14" />
   </joint>
-  <gazebo reference="hokuyo_link">
+  <gazebo reference="laser_frame">
     <material>Gazebo/Black</material>
     <sensor type="ray" name="head_hokuyo_sensor">
@@ -246,5 +257,5 @@
       <plugin name="gazebo_ros_head_hokuyo_controller" filename="libgazebo_ros_laser.so">
         <topicName>scan</topicName>
-        <frameName>hokuyo_link</frameName>
+        <frameName>laser_frame</frameName>
       </plugin>
     </sensor>

Commit message: [ROS] wr8_description fixed TF collision in model, wip fixing model rendering

File: wr8_description/urdf/model.urdf.xacro (robot description, xacro)
@@ -130,5 +130,5 @@
       <axis xyz="0 0 -1"/>
     </joint>
-<!--     <transmission name="${name}_rotate_trans">
+    <!-- <transmission name="${name}_rotate_trans">
       <type>transmission_interface/SimpleTransmission</type>
       <joint name="${name}_rotate_joint">
@@ -173,14 +173,14 @@
     <!-- </visual> -->
   </gazebo>
-  <joint name="base_footage_2_link" type="fixed">
-    <parent link="base_footprint"/>
-    <child link="base_link"/>
+  <joint name="base_link_2_footprint" type="fixed">
+    <parent link="base_link"/>
+    <child link="base_footprint"/>
     <!-- base_footprint - base_link on floor -->
-    <origin xyz="0 0 ${wheel_radius}" rpy="0 0 0"/>
+    <origin xyz="0 0 ${-wheel_radius}" rpy="0 0 0"/>
   </joint>
-  <joint name="base_footage_2_center" type="fixed">
-    <parent link="base_footprint"/>
+  <joint name="base_link_2_center" type="fixed">
+    <parent link="base_link"/>
     <child link="base_center"/>
-    <origin xyz="${wheelbase/2} 0 ${wheel_radius}" rpy="0 0 0"/>
+    <origin xyz="${wheelbase/2} 0 0" rpy="0 0 0"/>
   </joint>
 <!--
@@ -188,6 +188,8 @@
   <xacro:steering_wheel name="left_steer_wheel" base_name="base_center" xyz="${wheelbase/2} ${chassis_width/2} 0" ref="1" />
  -->
-  <xacro:steering_wheel name="right_steer_wheel" base_name="base_center" xyz="${wheelbase/2} ${-(chassis_width/2 + wheel_chassis_bias)} ${-chassis_height/2}" ref="-1" />
-  <xacro:steering_wheel name="left_steer_wheel" base_name="base_center" xyz="${wheelbase/2} ${(chassis_width/2 + wheel_chassis_bias)} ${-chassis_height/2}" ref="1" />
+  <xacro:steering_wheel name="right_steer_wheel" base_name="base_center"
+                        xyz="${wheelbase/2} ${-(chassis_width/2 + wheel_chassis_bias)} ${-chassis_height/2}" ref="-1" />
+  <xacro:steering_wheel name="left_steer_wheel" base_name="base_center"
+                        xyz="${wheelbase/2} ${(chassis_width/2 + wheel_chassis_bias)} ${-chassis_height/2}" ref="1" />
   <xacro:traveling_wheel name="right_travel_wheel" base_name="base_center"
                          xyz="${-wheelbase/2} ${-(chassis_width/2 + wheel_chassis_bias)} ${-chassis_height/2}" />
@@ -222,5 +224,5 @@
     </visual>
   </link>
-  <joint name="hokuyo_joint" type="fixed">
+  <joint name="laser_joint" type="fixed">
     <child link="laser_frame" />
     <parent link="base_link" />

Commit message: [ROS/gazebo] New model representation

File: wr8_description/urdf/model.urdf.xacro (robot description, xacro)
@@ -5,4 +5,9 @@
   <xacro:property name="wheel_mass" value="0.056" />
   <xacro:property name="wheel_chassis_bias" value="${wheel_width/2}" />
+  <!-- Just to be visible =) -->
+  <xacro:property name="lidar_height" value="0.02"/>
+  <xacro:property name="lidar_radius" value="0.04"/>
+  <!-- Taken from physical parameters (wr8_software/launch/base/lidar.launch) -->
+  <xacro:property name="base_link_2_laser_xyz" value="0.14 0 0.14" />
   <xacro:property name="chassis_mass" value="3.7" />
   <xacro:property name="chassis_length" value="0.485" />
@@ -10,4 +15,6 @@
   <xacro:property name="chassis_height" value="0.05" />
   <xacro:property name="wheelbase" value="0.3" />
+  <xacro:property name="half_wheelbase" value="${wheelbase/2}" />
+  <xacro:property name="half_track_width" value="${(chassis_width/2 + wheel_chassis_bias)}" />
   <xacro:property name="lidar_mass" value="0.1" />
   <!-- https://github.com/jbpassot/ackermann_vehicle/blob/master/ackermann_vehicle_description/urdf/em_3905.urdf.xacro -->
@@ -18,6 +25,35 @@
   <xacro:property name="wheel_turn_limit" value="${degrees_30}"/>
   <!-- <xacro:property name="servo_stall_torque" value="0.5649"/> -->
-  <xacro:property name="servo_stall_torque" value="100"/>
-  <xacro:property name="servo_no_load_speed" value="4.553"/>
+  <!-- <xacro:property name="servo_stall_torque" value="100"/>
+  <xacro:property name="servo_no_load_speed" value="4.553"/> -->
+  <xacro:property name="wheel_friction" value="1.75" />
+  <xacro:arg name="pub_tf" default="true" />
+  <xacro:arg name="robot_name" default="robot" />
+  <!-- Gazebo plugins -->
+  <gazebo>
+    <!-- <plugin name="gazebo_ros_control" filename="libgazebo_ros_control.so">
+      <robotNamespace>/</robotNamespace>
+    </plugin> -->
+    <!-- Simulated vehicle interface -->
+    <plugin name="wr8_interface_plugin" filename="libwr8_interface_plugin.so" >
+      <robotName>$(arg robot_name)</robotName>
+      <pubTf>$(arg pub_tf)</pubTf>
+      <tfFreq>100.0</tfFreq>
+    </plugin>
+    <!-- Publish current joint angles -->
+    <plugin name="joint_state_publisher" filename="libgazebo_ros_joint_state_publisher.so">
+        <robotNamespace>$(arg robot_name)</robotNamespace>
+        <jointName>
+            fl_steer_joint,
+            fr_steer_joint,
+            fl_speed_joint,
+            fr_speed_joint,
+            rl_speed_joint,
+            rr_speed_joint
+        </jointName>
+        <updateRate>100</updateRate>
+        <alwaysOn>true</alwaysOn>
+    </plugin>
+  </gazebo>
   <!-- INERTIAL MACROS -->
   <xacro:macro name="null_inertial">
@@ -73,70 +109,40 @@
     </link>
     <gazebo reference="${name}">
-      <mu1>1.0</mu1>
-      <mu2>1.0</mu2>
-      <kp>10000000</kp>
-      <kd>1</kd>
-      <!-- <minDepth>0.01</minDepth> -->
-      <!-- <maxVel>10.0</maxVel>  -->
+      <mu1>${wheel_friction}</mu1>
+      <mu2>${wheel_friction}</mu2>
       <material>Gazebo/Black</material>
     </gazebo>
   </xacro:macro>
-  <xacro:macro name="traveling_wheel" params="name base_name xyz ">
-    <xacro:wheel_object name="${name}" />
-    <joint name="${name}_rotate_joint" type="continuous">
+  <xacro:macro name="speed_wheel" params="name base_name xyz ">
+    <xacro:wheel_object name="wheel_${name}" />
+    <joint name="${name}_speed_joint" type="continuous">
       <parent link="${base_name}"/>
-      <child link="${name}"/>
+      <child link="wheel_${name}"/>
       <origin xyz="${xyz}" rpy="${pi/2} 0 0"/>
       <axis xyz="0 0 -1"/>
+      <limit effort="1000.0" velocity="22.0" />
     </joint>
-    <transmission name="${name}_rotate_trans">
-      <type>transmission_interface/SimpleTransmission</type>
-      <joint name="${name}_rotate_joint">
-        <hardwareInterface>hardware_interface/VelocityJointInterface</hardwareInterface>
-      </joint>
-      <actuator name="${name}_rotate_motor">
-        <mechanicalReduction>1</mechanicalReduction>
-      </actuator>
-    </transmission>
-  </xacro:macro>
-  <xacro:macro name="steering_wheel" params="name base_name xyz ref">
-    <link name="${name}_base">
+  </xacro:macro>
+  <xacro:macro name="steer_wheel" params="name base_name xyz">
+    <xacro:wheel_object name="wheel_${name}" />
+    <link name="steer_${name}">
       <xacro:null_inertial/>
     </link>
-    <joint name="${name}_steering_joint" type="revolute">
-      <limit lower="${-wheel_turn_limit}" upper="${wheel_turn_limit}"
-             effort="${servo_stall_torque}" velocity="${servo_no_load_speed}"/>
+    <joint name="${name}_steer_joint" type="revolute">
+      <limit lower="${-wheel_turn_limit}"
+             upper="${wheel_turn_limit}"
+             effort="0" velocity="0"/>
       <parent link="${base_name}"/>
-      <child link="${name}_base"/>
+      <child link="steer_${name}"/>
       <origin xyz="${xyz}" rpy="0 0 0"/>
       <axis xyz="0 0 1"/>
     </joint>
-    <transmission name="${name}_steer_trans">
-      <type>transmission_interface/SimpleTransmission</type>
-      <joint name="${name}_steering_joint">
-        <hardwareInterface>hardware_interface/PositionJointInterface</hardwareInterface>
-      </joint>
-      <actuator name="${name}_steering_motor">
-        <mechanicalReduction>1</mechanicalReduction>
-      </actuator>
-    </transmission>
-    <!-- <xacro:traveling_wheel name="${name}" base_name="${name}_base" xyz="0 ${ref * wheel_chassis_bias} 0" /> -->
-    <!-- <xacro:traveling_wheel name="${name}" base_name="${name}_base" xyz="0 0 0" /> -->
-    <xacro:wheel_object name="${name}" />
-    <joint name="${name}_rotate_joint" type="continuous">
-      <parent link="${name}_base"/>
-      <child link="${name}"/>
+    <joint name="${name}_speed_joint" type="continuous">
+      <parent link="steer_${name}"/>
+      <child link="wheel_${name}"/>
       <origin xyz="0 0 0" rpy="${pi/2} 0 0"/>
       <axis xyz="0 0 -1"/>
+      <limit effort="1000.0" velocity="22.0" />
     </joint>
-    <!-- <transmission name="${name}_rotate_trans">
-      <type>transmission_interface/SimpleTransmission</type>
-      <joint name="${name}_rotate_joint">
-        <hardwareInterface>hardware_interface/VelocityJointInterface</hardwareInterface>
-      </joint>
-      <actuator name="${name}_rotate_motor">
-        <mechanicalReduction>1</mechanicalReduction>
-      </actuator>
-    </transmission> -->
   </xacro:macro>
   <!-- base_footprint - base_link on floor -->
@@ -167,15 +173,11 @@
   </link>
   <gazebo reference="base_center">
-    <!-- <visual>   -->
-      <material>
-        Gazebo/Orange
-      </material>
-    <!-- </visual> -->
+      <material>Gazebo/Orange</material>
   </gazebo>
-  <joint name="base_link_2_footprint" type="fixed">
-    <parent link="base_link"/>
-    <child link="base_footprint"/>
+  <joint name="base_footprint_2_link" type="fixed">
+    <parent link="base_footprint"/>
+    <child link="base_link"/>
     <!-- base_footprint - base_link on floor -->
-    <origin xyz="0 0 ${-wheel_radius}" rpy="0 0 0"/>
+    <origin xyz="0 0 ${wheel_radius}" rpy="0 0 0"/>
   </joint>
   <joint name="base_link_2_center" type="fixed">
@@ -184,25 +186,13 @@
     <origin xyz="${wheelbase/2} 0 0" rpy="0 0 0"/>
   </joint>
-<!--
-  <xacro:steering_wheel name="right_steer_wheel" base_name="base_center" xyz="${wheelbase/2} ${-chassis_width/2} 0" ref="-1" />
-  <xacro:steering_wheel name="left_steer_wheel" base_name="base_center" xyz="${wheelbase/2} ${chassis_width/2} 0" ref="1" />
- -->
-  <xacro:steering_wheel name="right_steer_wheel" base_name="base_center"
-                        xyz="${wheelbase/2} ${-(chassis_width/2 + wheel_chassis_bias)} ${-chassis_height/2}" ref="-1" />
-  <xacro:steering_wheel name="left_steer_wheel" base_name="base_center"
-                        xyz="${wheelbase/2} ${(chassis_width/2 + wheel_chassis_bias)} ${-chassis_height/2}" ref="1" />
-  <xacro:traveling_wheel name="right_travel_wheel" base_name="base_center"
-                         xyz="${-wheelbase/2} ${-(chassis_width/2 + wheel_chassis_bias)} ${-chassis_height/2}" />
-  <xacro:traveling_wheel name="left_travel_wheel" base_name="base_center"
-                         xyz="${-wheelbase/2} ${(chassis_width/2 + wheel_chassis_bias)} ${-chassis_height/2}" />
-  <!-- Gazebo plugin for ROS Control -->
-  <gazebo>
-    <plugin name="gazebo_ros_control" filename="libgazebo_ros_control.so">
-      <!-- <robotNamespace>/</robotNamespace> -->
-    </plugin>
-  </gazebo>
+  <xacro:speed_wheel name="rl" base_name="base_center"
+                     xyz="${-half_wheelbase} ${-half_track_width} ${-chassis_height/2}" />
+  <xacro:speed_wheel name="rr" base_name="base_center"
+                     xyz="${-half_wheelbase} ${half_track_width} ${-chassis_height/2}" />
+  <xacro:steer_wheel name="fl" base_name="base_center"
+                     xyz="${half_wheelbase} ${-half_track_width} ${-chassis_height/2}" />
+  <xacro:steer_wheel name="fr" base_name="base_center"
+                     xyz="${half_wheelbase} ${half_track_width} ${-chassis_height/2}" />
   <!-- Setup LIDAR -->
-  <xacro:property name="lidar_height" value="0.04"/>
-  <xacro:property name="lidar_radius" value="0.04"/>
   <link name="laser_frame">
     <xacro:solid_cylinder_inertial
@@ -227,6 +217,5 @@
     <child link="laser_frame" />
     <parent link="base_link" />
-    <!-- Taken from physical parameters (wr8_software/launch/base/lidar.launch) -->
-    <origin xyz="0.14 0 0.14" />
+    <origin xyz="${base_link_2_laser_xyz}" />
   </joint>
   <gazebo reference="laser_frame">
@@ -247,5 +236,5 @@
         </scan>
         <range>
-          <min>0.10</min>
+          <min>0.15</min>
           <max>10.0</max>
           <resolution>0.01</resolution>

Commit message: [ROS/gazebo] Steering angle done

File: wr8_description/urdf/model.urdf.xacro (robot description, xacro)
@@ -19,9 +19,10 @@
   <xacro:property name="lidar_mass" value="0.1" />
   <!-- https://github.com/jbpassot/ackermann_vehicle/blob/master/ackermann_vehicle_description/urdf/em_3905.urdf.xacro -->
-  <xacro:property name="degrees_45" value="0.785398163"/>
-  <xacro:property name="degrees_90" value="1.57079633"/>
+  <xacro:property name="degrees_45" value="${pi/4}"/>
+  <xacro:property name="degrees_90" value="${pi/2}"/>
   <!-- ~0.5 rad -->
-  <xacro:property name="degrees_30" value="${pi/3}"/>
-  <xacro:property name="wheel_turn_limit" value="${degrees_30}"/>
+  <xacro:property name="degrees_30" value="${pi/6}"/>
+  <xacro:property name="mid_wheel_turn_limit" value="${degrees_30}"/>
+  <xacro:property name="wheel_turn_limit" value="${degrees_45}"/>
   <!-- <xacro:property name="servo_stall_torque" value="0.5649"/> -->
   <!-- <xacro:property name="servo_stall_torque" value="100"/>
@@ -40,4 +41,7 @@
       <pubTf>$(arg pub_tf)</pubTf>
       <tfFreq>100.0</tfFreq>
+      <maxSteerRad>${mid_wheel_turn_limit}</maxSteerRad>
+      <wheelbase>${wheelbase}</wheelbase>
+      <trackWidth>${half_track_width*2}</trackWidth>
     </plugin>
     <!-- Publish current joint angles -->
@@ -247,5 +251,5 @@
       </ray>
       <plugin name="gazebo_ros_head_hokuyo_controller" filename="libgazebo_ros_laser.so">
-        <topicName>scan</topicName>
+        <topicName>$(arg robot_name)/scan</topicName>
         <frameName>laser_frame</frameName>
       </plugin>

Commit message: Stereo camera + signs camera not tested

File: wr8_description/urdf/model.urdf.xacro (robot description, xacro)
@@ -19,6 +19,6 @@
   <xacro:property name="lidar_mass" value="0.1" />
   <!-- https://github.com/jbpassot/ackermann_vehicle/blob/master/ackermann_vehicle_description/urdf/em_3905.urdf.xacro -->
+  <xacro:property name="degrees_90" value="${pi/2}"/>
   <xacro:property name="degrees_45" value="${pi/4}"/>
-  <xacro:property name="degrees_90" value="${pi/2}"/>
   <!-- ~0.5 rad -->
   <xacro:property name="degrees_30" value="${pi/6}"/>
@@ -29,4 +29,10 @@
   <xacro:property name="servo_no_load_speed" value="4.553"/> -->
   <xacro:property name="wheel_friction" value="1.75" />
+  <!-- Stereo camera properties -->
+  <xacro:property name="camera_height" value="0.05"/>
+  <xacro:property name="camera_radius" value="0.02"/>
+  <xacro:property name="camera_mass" value="0.05"/>
+  <xacro:property name="stereo_base_link_lcam_xyz" value="0.14 0.15 0.18"/>
+  <xacro:property name="stereo_base_link_rcam_xyz" value="0.14 -0.15 0.18"/>
   <xacro:arg name="pub_tf" default="true" />
   <xacro:arg name="robot_name" default="robot" />
@@ -259,3 +265,71 @@
     </sensor>
   </gazebo>
+  <!-- Stereo camera macro -->
+  <xacro:macro name="single_camera" params="name xyz rpy">
+    <link name="${name}_frame">
+      <xacro:solid_cylinder_inertial
+          r="${camera_radius}" h="${camera_height}"
+          mass="${camera_mass}" >
+        <origin xyz="0 0 0" rpy="0 ${degrees_90} 0" />
+      </xacro:solid_cylinder_inertial>
+      <collision>
+        <origin xyz="0 0 0" rpy="0 ${degrees_90} 0" />
+        <geometry>
+          <cylinder length="${camera_height}" radius="${camera_radius}"/>
+        </geometry>
+      </collision>
+      <visual>
+        <origin xyz="0 0 0" rpy="0 ${degrees_90} 0" />
+        <geometry>
+          <cylinder length="${camera_height}" radius="${camera_radius}"/>
+        </geometry>
+      </visual>
+    </link>
+    <joint name="${name}_joint" type="fixed">
+      <child link="${name}_frame" />
+      <parent link="base_link" />
+      <origin xyz="${xyz}" rpy="${rpy}" />
+    </joint>
+    <gazebo reference="${name}_frame">
+      <material>Gazebo/Black</material>
+      <sensor type="camera" name="${name}">
+        <!-- required FPS -->
+        <update_rate>30.0</update_rate>
+        <camera name="${name}">
+          <horizontal_fov>1.3962634</horizontal_fov>
+          <image>
+            <width>800</width>
+            <height>800</height>
+            <format>R8G8B8</format>
+          </image>
+          <clip>
+            <near>0.02</near>
+            <far>300</far>
+          </clip>
+          <noise>
+            <type>gaussian</type>
+            <mean>0.0</mean>
+            <stddev>0.007</stddev>
+        </noise>
+        </camera>
+        <plugin name="${name}_controller" filename="libgazebo_ros_camera.so">
+          <alwaysOn>true</alwaysOn>
+          <updateRate>0.0</updateRate>
+          <cameraName>$(arg robot_name)/${name}</cameraName>
+          <imageTopicName>cam_image_raw</imageTopicName>
+          <cameraInfoTopicName>cam_info</cameraInfoTopicName>
+          <frameName>lcam_frame</frameName>
+          <hackBaseline>0.07</hackBaseline>
+          <distortionK1>0.0</distortionK1>
+          <distortionK2>0.0</distortionK2>
+          <distortionK3>0.0</distortionK3>
+          <distortionT1>0.0</distortionT1>
+          <distortionT2>0.0</distortionT2>
+        </plugin>
+      </sensor>
+    </gazebo>
+  </xacro:macro>
+  <xacro:single_camera name="lcam" xyz="${stereo_base_link_lcam_xyz}" rpy="0 0 0" />
+  <xacro:single_camera name="rcam" xyz="${stereo_base_link_rcam_xyz}" rpy="0 0 0" />
+  <xacro:single_camera name="signs_cam" xyz="1 0 1" rpy="0 ${degrees_30} 0" />
 </robot>
