Commit message: Steome fixes

File: wr8_description/urdf/model.urdf.xacro (robot description, xacro)
@@ -266,5 +266,5 @@
   </gazebo>
   <!-- Stereo camera macro -->
-  <xacro:macro name="single_camera" params="name xyz rpy">
+  <xacro:macro name="single_camera" params="name xyz rpy fov">
     <link name="${name}_frame">
       <xacro:solid_cylinder_inertial
@@ -297,8 +297,8 @@
         <update_rate>30.0</update_rate>
         <camera name="${name}">
-          <horizontal_fov>1.3962634</horizontal_fov>
+          <horizontal_fov>${fov}</horizontal_fov>
           <image>
             <width>800</width>
-            <height>800</height>
+            <height>600</height>
             <format>R8G8B8</format>
           </image>
@@ -311,5 +311,5 @@
             <mean>0.0</mean>
             <stddev>0.007</stddev>
-        </noise>
+          </noise>
         </camera>
         <plugin name="${name}_controller" filename="libgazebo_ros_camera.so">
@@ -317,8 +317,8 @@
           <updateRate>0.0</updateRate>
           <cameraName>$(arg robot_name)/${name}</cameraName>
-          <imageTopicName>cam_image_raw</imageTopicName>
-          <cameraInfoTopicName>cam_info</cameraInfoTopicName>
+          <imageTopicName>image_raw</imageTopicName>
+          <cameraInfoTopicName>camera_info</cameraInfoTopicName>
           <frameName>lcam_frame</frameName>
-          <hackBaseline>0.07</hackBaseline>
+          <hackBaseline>0.3</hackBaseline>
           <distortionK1>0.0</distortionK1>
           <distortionK2>0.0</distortionK2>
@@ -330,6 +330,6 @@
     </gazebo>
   </xacro:macro>
-  <xacro:single_camera name="lcam" xyz="${stereo_base_link_lcam_xyz}" rpy="0 0 0" />
-  <xacro:single_camera name="rcam" xyz="${stereo_base_link_rcam_xyz}" rpy="0 0 0" />
-  <xacro:single_camera name="signs_cam" xyz="1 0 1" rpy="0 ${degrees_30} 0" />
+  <xacro:single_camera name="left_cam" xyz="${stereo_base_link_lcam_xyz}" rpy="0 0 0" fov="1.3962634" />
+  <xacro:single_camera name="right_cam" xyz="${stereo_base_link_rcam_xyz}" rpy="0 0 0" fov="1.3962634" />
+  <xacro:single_camera name="signs_cam" xyz="1 0 1" rpy="0 ${degrees_30} 0" fov="2.094" />
 </robot>

Commit message: Stereo camera with processing done

File: wr8_description/urdf/model.urdf.xacro (robot description, xacro)
@@ -33,6 +33,6 @@
   <xacro:property name="camera_radius" value="0.02"/>
   <xacro:property name="camera_mass" value="0.05"/>
-  <xacro:property name="stereo_base_link_lcam_xyz" value="0.14 0.15 0.18"/>
-  <xacro:property name="stereo_base_link_rcam_xyz" value="0.14 -0.15 0.18"/>
+  <xacro:property name="stereo_base_link_lcam_xyz" value="0.05 0.035 0.18"/>
+  <xacro:property name="stereo_base_link_rcam_xyz" value="0.05 -0.035 0.18"/>
   <xacro:arg name="pub_tf" default="true" />
   <xacro:arg name="robot_name" default="robot" />
@@ -265,6 +265,6 @@
     </sensor>
   </gazebo>
-  <!-- Stereo camera macro -->
-  <xacro:macro name="single_camera" params="name xyz rpy fov">
+  <!-- Camera link -->
+  <xacro:macro name="camera_link" params="name">
     <link name="${name}_frame">
       <xacro:solid_cylinder_inertial
@@ -286,7 +286,11 @@
       </visual>
     </link>
+  </xacro:macro>
+  <!-- Single camera macro -->
+  <xacro:macro name="single_camera" params="name xyz rpy fov">
+    <xacro:camera_link name="${name}" />
     <joint name="${name}_joint" type="fixed">
       <child link="${name}_frame" />
-      <parent link="base_link" />
+      <parent link="base_center" />
       <origin xyz="${xyz}" rpy="${rpy}" />
     </joint>
@@ -294,7 +298,64 @@
       <material>Gazebo/Black</material>
       <sensor type="camera" name="${name}">
-        <!-- required FPS -->
         <update_rate>30.0</update_rate>
         <camera name="${name}">
+          <horizontal_fov>${fov}</horizontal_fov>
+          <image>
+            <width>800</width>
+            <height>600</height>
+            <format>R8G8B8</format>
+          </image>
+          <clip>
+            <near>0.02</near>
+            <far>300</far>
+          </clip>
+          <noise>
+            <type>gaussian</type>
+            <mean>0.0</mean>
+            <stddev>0.001</stddev>
+          </noise>
+        </camera>
+        <plugin name="${name}_controller" filename="libgazebo_ros_camera.so">
+          <alwaysOn>true</alwaysOn>
+          <updateRate>30.0</updateRate>
+          <cameraName>$(arg robot_name)/${name}</cameraName>
+          <imageTopicName>image_raw</imageTopicName>
+          <cameraInfoTopicName>camera_info</cameraInfoTopicName>
+          <frameName>${name}_frame</frameName>
+          <hackBaseline>0.07</hackBaseline>
+          <distortionK1>0.0</distortionK1>
+          <distortionK2>0.0</distortionK2>
+          <distortionK3>0.0</distortionK3>
+          <distortionT1>0.0</distortionT1>
+          <distortionT2>0.0</distortionT2>
+        </plugin>
+      </sensor>
+    </gazebo>
+  </xacro:macro>
+  <!-- Stereo camera macro -->
+  <xacro:macro name="stereo_camera" params="name fov">
+    <xacro:camera_link name="${name}_left" />
+    <xacro:camera_link name="${name}_right" />
+    <joint name="${name}_left_joint" type="fixed">
+      <child link="${name}_left_frame" />
+      <parent link="base_center" />
+      <origin xyz="${stereo_base_link_lcam_xyz}" rpy="0 0 0" />
+    </joint>
+    <joint name="${name}_right_joint" type="fixed">
+      <child link="${name}_right_frame" />
+      <parent link="base_center" />
+      <origin xyz="${stereo_base_link_rcam_xyz}" rpy="0 0 0" />
+    </joint>
+    <link name="${name}_left_optical_frame"/>
+    <joint name="${name}_left_optical_frame_joint" type="fixed">
+      <origin xyz="0 0 0" rpy="-${degrees_90} 0.0 -${degrees_90}" />
+      <parent link="${name}_left_frame" />
+      <child link="${name}_left_optical_frame"/>
+    </joint>
+    <gazebo reference="${name}_left_frame">
+      <material>Gazebo/Black</material>
+      <sensor type="multicamera" name="${name}">
+        <update_rate>30.0</update_rate>
+        <camera name="left">
           <horizontal_fov>${fov}</horizontal_fov>
           <image>
@@ -313,12 +374,31 @@
           </noise>
         </camera>
-        <plugin name="${name}_controller" filename="libgazebo_ros_camera.so">
+        <camera name="right">
+          <pose>0 -0.07 0 0 0 0</pose>
+          <!-- <pose>0 -0.035 0 0 0 0</pose> -->
+          <horizontal_fov>${fov}</horizontal_fov>
+          <image>
+            <width>800</width>
+            <height>600</height>
+            <format>R8G8B8</format>
+          </image>
+          <clip>
+            <near>0.02</near>
+            <far>300</far>
+          </clip>
+          <noise>
+            <type>gaussian</type>
+            <mean>0.0</mean>
+            <stddev>0.007</stddev>
+          </noise>
+        </camera>
+        <plugin name="${name}_controller" filename="libgazebo_ros_multicamera.so">
           <alwaysOn>true</alwaysOn>
-          <updateRate>0.0</updateRate>
+          <updateRate>30.0</updateRate>
           <cameraName>$(arg robot_name)/${name}</cameraName>
           <imageTopicName>image_raw</imageTopicName>
           <cameraInfoTopicName>camera_info</cameraInfoTopicName>
-          <frameName>lcam_frame</frameName>
-          <hackBaseline>0.3</hackBaseline>
+          <frameName>${name}_left_optical_frame</frameName>
+          <hackBaseline>0.07</hackBaseline>
           <distortionK1>0.0</distortionK1>
           <distortionK2>0.0</distortionK2>
@@ -330,6 +410,5 @@
     </gazebo>
   </xacro:macro>
-  <xacro:single_camera name="left_cam" xyz="${stereo_base_link_lcam_xyz}" rpy="0 0 0" fov="1.3962634" />
-  <xacro:single_camera name="right_cam" xyz="${stereo_base_link_rcam_xyz}" rpy="0 0 0" fov="1.3962634" />
-  <xacro:single_camera name="signs_cam" xyz="1 0 1" rpy="0 ${degrees_30} 0" fov="2.094" />
+  <xacro:stereo_camera name="stereo_camera" fov="1.3962634" />
+  <xacro:single_camera name="signs_camera" xyz="-0.05 0 0.2" rpy="0 -${degrees_30} -${degrees_30}" fov="2.094" />
 </robot>

Commit message: Signs camera prepared - test required

File: wr8_description/urdf/model.urdf.xacro (robot description, xacro)
@@ -295,4 +295,10 @@
       <origin xyz="${xyz}" rpy="${rpy}" />
     </joint>
+    <link name="${name}_optical_frame"/>
+    <joint name="${name}_optical_frame_joint" type="fixed">
+      <origin xyz="0 0 0" rpy="-${degrees_90} 0.0 -${degrees_90}" />
+      <parent link="${name}_frame" />
+      <child link="${name}_optical_frame"/>
+    </joint>
     <gazebo reference="${name}_frame">
       <material>Gazebo/Black</material>
@@ -322,5 +328,5 @@
           <imageTopicName>image_raw</imageTopicName>
           <cameraInfoTopicName>camera_info</cameraInfoTopicName>
-          <frameName>${name}_frame</frameName>
+          <frameName>${name}_optical_frame</frameName>
           <hackBaseline>0.07</hackBaseline>
           <distortionK1>0.0</distortionK1>
@@ -411,4 +417,5 @@
   </xacro:macro>
   <xacro:stereo_camera name="stereo_camera" fov="1.3962634" />
-  <xacro:single_camera name="signs_camera" xyz="-0.05 0 0.2" rpy="0 -${degrees_30} -${degrees_30}" fov="2.094" />
+  <!-- <xacro:single_camera name="signs_camera" xyz="-0.05 0 0.2" rpy="0 -${degrees_30} -${degrees_30}" fov="2.094" /> -->
+  <xacro:single_camera name="signs_camera" xyz="-0.05 0 0.3" rpy="0 -${degrees_30} -${degrees_30}" fov="1.3962634" />
 </robot>

Commit message: Refactoring + stereo frames and scripts fixed

File: wr8_description/urdf/model.urdf.xacro (robot description, xacro)
@@ -36,5 +36,5 @@
   <xacro:property name="stereo_base_link_rcam_xyz" value="0.05 -0.035 0.18"/>
   <xacro:arg name="pub_tf" default="true" />
-  <xacro:arg name="robot_name" default="robot" />
+  <xacro:arg name="robot_name" default="" />
   <!-- Gazebo plugins -->
   <gazebo>
@@ -353,9 +353,9 @@
       <origin xyz="${stereo_base_link_rcam_xyz}" rpy="0 0 0" />
     </joint>
-    <link name="${name}_left_optical_frame"/>
-    <joint name="${name}_left_optical_frame_joint" type="fixed">
+    <link name="${name}_optical_frame"/>
+    <joint name="${name}_optical_frame_joint" type="fixed">
       <origin xyz="0 0 0" rpy="-${degrees_90} 0.0 -${degrees_90}" />
       <parent link="${name}_left_frame" />
-      <child link="${name}_left_optical_frame"/>
+      <child link="${name}_optical_frame"/>
     </joint>
     <gazebo reference="${name}_left_frame">
@@ -405,5 +405,5 @@
           <imageTopicName>image_raw</imageTopicName>
           <cameraInfoTopicName>camera_info</cameraInfoTopicName>
-          <frameName>${name}_left_optical_frame</frameName>
+          <frameName>${name}_optical_frame</frameName>
           <hackBaseline>0.07</hackBaseline>
           <distortionK1>0.0</distortionK1>

Commit message: [ROS common] add stereo switcher

File: wr8_description/urdf/model.urdf.xacro (robot description, xacro)
@@ -37,4 +37,5 @@
   <xacro:arg name="pub_tf" default="true" />
   <xacro:arg name="robot_name" default="" />
+  <xacro:arg name="enable_stereo" default="true" />
   <!-- Gazebo plugins -->
   <gazebo>
@@ -265,157 +266,158 @@
     </sensor>
   </gazebo>
-  <!-- Camera link -->
-  <xacro:macro name="camera_link" params="name">
-    <link name="${name}_frame">
-      <xacro:solid_cylinder_inertial
-          r="${camera_radius}" h="${camera_height}"
-          mass="${camera_mass}" >
-        <origin xyz="0 0 0" rpy="0 ${degrees_90} 0" />
-      </xacro:solid_cylinder_inertial>
-      <collision>
-        <origin xyz="0 0 0" rpy="0 ${degrees_90} 0" />
-        <geometry>
-          <cylinder length="${camera_height}" radius="${camera_radius}"/>
-        </geometry>
-      </collision>
-      <visual>
-        <origin xyz="0 0 0" rpy="0 ${degrees_90} 0" />
-        <geometry>
-          <cylinder length="${camera_height}" radius="${camera_radius}"/>
-        </geometry>
-      </visual>
-    </link>
-  </xacro:macro>
-  <!-- Single camera macro -->
-  <xacro:macro name="single_camera" params="name xyz rpy fov">
-    <xacro:camera_link name="${name}" />
-    <joint name="${name}_joint" type="fixed">
-      <child link="${name}_frame" />
-      <parent link="base_center" />
-      <origin xyz="${xyz}" rpy="${rpy}" />
-    </joint>
-    <link name="${name}_optical_frame"/>
-    <joint name="${name}_optical_frame_joint" type="fixed">
-      <origin xyz="0 0 0" rpy="-${degrees_90} 0.0 -${degrees_90}" />
-      <parent link="${name}_frame" />
-      <child link="${name}_optical_frame"/>
-    </joint>
-    <gazebo reference="${name}_frame">
-      <material>Gazebo/Black</material>
-      <sensor type="camera" name="${name}">
-        <update_rate>30.0</update_rate>
-        <camera name="${name}">
-          <horizontal_fov>${fov}</horizontal_fov>
-          <image>
-            <width>800</width>
-            <height>600</height>
-            <format>R8G8B8</format>
-          </image>
-          <clip>
-            <near>0.02</near>
-            <far>300</far>
-          </clip>
-          <noise>
-            <type>gaussian</type>
-            <mean>0.0</mean>
-            <stddev>0.001</stddev>
-          </noise>
-        </camera>
-        <plugin name="${name}_controller" filename="libgazebo_ros_camera.so">
-          <alwaysOn>true</alwaysOn>
-          <updateRate>30.0</updateRate>
-          <cameraName>$(arg robot_name)/${name}</cameraName>
-          <imageTopicName>image_raw</imageTopicName>
-          <cameraInfoTopicName>camera_info</cameraInfoTopicName>
-          <frameName>${name}_optical_frame</frameName>
-          <hackBaseline>0.07</hackBaseline>
-          <distortionK1>0.0</distortionK1>
-          <distortionK2>0.0</distortionK2>
-          <distortionK3>0.0</distortionK3>
-          <distortionT1>0.0</distortionT1>
-          <distortionT2>0.0</distortionT2>
-        </plugin>
-      </sensor>
-    </gazebo>
-  </xacro:macro>
-  <!-- Stereo camera macro -->
-  <xacro:macro name="stereo_camera" params="name fov">
-    <xacro:camera_link name="${name}_left" />
-    <xacro:camera_link name="${name}_right" />
-    <joint name="${name}_left_joint" type="fixed">
-      <child link="${name}_left_frame" />
-      <parent link="base_center" />
-      <origin xyz="${stereo_base_link_lcam_xyz}" rpy="0 0 0" />
-    </joint>
-    <joint name="${name}_right_joint" type="fixed">
-      <child link="${name}_right_frame" />
-      <parent link="base_center" />
-      <origin xyz="${stereo_base_link_rcam_xyz}" rpy="0 0 0" />
-    </joint>
-    <link name="${name}_optical_frame"/>
-    <joint name="${name}_optical_frame_joint" type="fixed">
-      <origin xyz="0 0 0" rpy="-${degrees_90} 0.0 -${degrees_90}" />
-      <parent link="${name}_left_frame" />
-      <child link="${name}_optical_frame"/>
-    </joint>
-    <gazebo reference="${name}_left_frame">
-      <material>Gazebo/Black</material>
-      <sensor type="multicamera" name="${name}">
-        <update_rate>30.0</update_rate>
-        <camera name="left">
-          <horizontal_fov>${fov}</horizontal_fov>
-          <image>
-            <width>800</width>
-            <height>600</height>
-            <format>R8G8B8</format>
-          </image>
-          <clip>
-            <near>0.02</near>
-            <far>300</far>
-          </clip>
-          <noise>
-            <type>gaussian</type>
-            <mean>0.0</mean>
-            <stddev>0.007</stddev>
-          </noise>
-        </camera>
-        <camera name="right">
-          <pose>0 -0.07 0 0 0 0</pose>
-          <!-- <pose>0 -0.035 0 0 0 0</pose> -->
-          <horizontal_fov>${fov}</horizontal_fov>
-          <image>
-            <width>800</width>
-            <height>600</height>
-            <format>R8G8B8</format>
-          </image>
-          <clip>
-            <near>0.02</near>
-            <far>300</far>
-          </clip>
-          <noise>
-            <type>gaussian</type>
-            <mean>0.0</mean>
-            <stddev>0.007</stddev>
-          </noise>
-        </camera>
-        <plugin name="${name}_controller" filename="libgazebo_ros_multicamera.so">
-          <alwaysOn>true</alwaysOn>
-          <updateRate>30.0</updateRate>
-          <cameraName>$(arg robot_name)/${name}</cameraName>
-          <imageTopicName>image_raw</imageTopicName>
-          <cameraInfoTopicName>camera_info</cameraInfoTopicName>
-          <frameName>${name}_optical_frame</frameName>
-          <hackBaseline>0.07</hackBaseline>
-          <distortionK1>0.0</distortionK1>
-          <distortionK2>0.0</distortionK2>
-          <distortionK3>0.0</distortionK3>
-          <distortionT1>0.0</distortionT1>
-          <distortionT2>0.0</distortionT2>
-        </plugin>
-      </sensor>
-    </gazebo>
-  </xacro:macro>
-  <xacro:stereo_camera name="stereo_camera" fov="1.3962634" />
-  <!-- <xacro:single_camera name="signs_camera" xyz="-0.05 0 0.2" rpy="0 -${degrees_30} -${degrees_30}" fov="2.094" /> -->
-  <xacro:single_camera name="signs_camera" xyz="-0.05 0 0.3" rpy="0 -${degrees_30} -${degrees_30}" fov="1.3962634" />
+  <xacro:if value="$(arg enable_stereo)">
+    <!-- Camera link -->
+    <xacro:macro name="camera_link" params="name">
+      <link name="${name}_frame">
+        <xacro:solid_cylinder_inertial
+            r="${camera_radius}" h="${camera_height}"
+            mass="${camera_mass}" >
+          <origin xyz="0 0 0" rpy="0 ${degrees_90} 0" />
+        </xacro:solid_cylinder_inertial>
+        <collision>
+          <origin xyz="0 0 0" rpy="0 ${degrees_90} 0" />
+          <geometry>
+            <cylinder length="${camera_height}" radius="${camera_radius}"/>
+          </geometry>
+        </collision>
+        <visual>
+          <origin xyz="0 0 0" rpy="0 ${degrees_90} 0" />
+          <geometry>
+            <cylinder length="${camera_height}" radius="${camera_radius}"/>
+          </geometry>
+        </visual>
+      </link>
+    </xacro:macro>
+    <!-- Single camera macro -->
+    <xacro:macro name="single_camera" params="name xyz rpy fov">
+      <xacro:camera_link name="${name}" />
+      <joint name="${name}_joint" type="fixed">
+        <child link="${name}_frame" />
+        <parent link="base_center" />
+        <origin xyz="${xyz}" rpy="${rpy}" />
+      </joint>
+      <link name="${name}_optical_frame"/>
+      <joint name="${name}_optical_frame_joint" type="fixed">
+        <origin xyz="0 0 0" rpy="-${degrees_90} 0.0 -${degrees_90}" />
+        <parent link="${name}_frame" />
+        <child link="${name}_optical_frame"/>
+      </joint>
+      <gazebo reference="${name}_frame">
+        <material>Gazebo/Black</material>
+        <sensor type="camera" name="${name}">
+          <update_rate>30.0</update_rate>
+          <camera name="${name}">
+            <horizontal_fov>${fov}</horizontal_fov>
+            <image>
+              <width>800</width>
+              <height>600</height>
+              <format>R8G8B8</format>
+            </image>
+            <clip>
+              <near>0.02</near>
+              <far>300</far>
+            </clip>
+            <noise>
+              <type>gaussian</type>
+              <mean>0.0</mean>
+              <stddev>0.001</stddev>
+            </noise>
+          </camera>
+          <plugin name="${name}_controller" filename="libgazebo_ros_camera.so">
+            <alwaysOn>true</alwaysOn>
+            <updateRate>30.0</updateRate>
+            <cameraName>$(arg robot_name)/${name}</cameraName>
+            <imageTopicName>image_raw</imageTopicName>
+            <cameraInfoTopicName>camera_info</cameraInfoTopicName>
+            <frameName>${name}_optical_frame</frameName>
+            <hackBaseline>0.07</hackBaseline>
+            <distortionK1>0.0</distortionK1>
+            <distortionK2>0.0</distortionK2>
+            <distortionK3>0.0</distortionK3>
+            <distortionT1>0.0</distortionT1>
+            <distortionT2>0.0</distortionT2>
+          </plugin>
+        </sensor>
+      </gazebo>
+    </xacro:macro>
+    <!-- Stereo camera macro -->
+    <xacro:macro name="stereo_camera" params="name fov">
+      <xacro:camera_link name="${name}_left" />
+      <xacro:camera_link name="${name}_right" />
+      <joint name="${name}_left_joint" type="fixed">
+        <child link="${name}_left_frame" />
+        <parent link="base_center" />
+        <origin xyz="${stereo_base_link_lcam_xyz}" rpy="0 0 0" />
+      </joint>
+      <joint name="${name}_right_joint" type="fixed">
+        <child link="${name}_right_frame" />
+        <parent link="base_center" />
+        <origin xyz="${stereo_base_link_rcam_xyz}" rpy="0 0 0" />
+      </joint>
+      <link name="${name}_optical_frame"/>
+      <joint name="${name}_optical_frame_joint" type="fixed">
+        <origin xyz="0 0 0" rpy="-${degrees_90} 0.0 -${degrees_90}" />
+        <parent link="${name}_left_frame" />
+        <child link="${name}_optical_frame"/>
+      </joint>
+      <gazebo reference="${name}_left_frame">
+        <material>Gazebo/Black</material>
+        <sensor type="multicamera" name="${name}">
+          <update_rate>30.0</update_rate>
+          <camera name="left">
+            <horizontal_fov>${fov}</horizontal_fov>
+            <image>
+              <width>800</width>
+              <height>600</height>
+              <format>R8G8B8</format>
+            </image>
+            <clip>
+              <near>0.02</near>
+              <far>300</far>
+            </clip>
+            <noise>
+              <type>gaussian</type>
+              <mean>0.0</mean>
+              <stddev>0.007</stddev>
+            </noise>
+          </camera>
+          <camera name="right">
+            <pose>0 -0.07 0 0 0 0</pose>
+            <!-- <pose>0 -0.035 0 0 0 0</pose> -->
+            <horizontal_fov>${fov}</horizontal_fov>
+            <image>
+              <width>800</width>
+              <height>600</height>
+              <format>R8G8B8</format>
+            </image>
+            <clip>
+              <near>0.02</near>
+              <far>300</far>
+            </clip>
+            <noise>
+              <type>gaussian</type>
+              <mean>0.0</mean>
+              <stddev>0.007</stddev>
+            </noise>
+          </camera>
+          <plugin name="${name}_controller" filename="libgazebo_ros_multicamera.so">
+            <alwaysOn>true</alwaysOn>
+            <updateRate>30.0</updateRate>
+            <cameraName>$(arg robot_name)/${name}</cameraName>
+            <imageTopicName>image_raw</imageTopicName>
+            <cameraInfoTopicName>camera_info</cameraInfoTopicName>
+            <frameName>${name}_optical_frame</frameName>
+            <hackBaseline>0.07</hackBaseline>
+            <distortionK1>0.0</distortionK1>
+            <distortionK2>0.0</distortionK2>
+            <distortionK3>0.0</distortionK3>
+            <distortionT1>0.0</distortionT1>
+            <distortionT2>0.0</distortionT2>
+          </plugin>
+        </sensor>
+      </gazebo>
+    </xacro:macro>
+    <xacro:stereo_camera name="stereo_camera" fov="1.3962634" />
+    <xacro:single_camera name="signs_camera" xyz="-0.05 0 0.3" rpy="0 -${degrees_30} -${degrees_30}" fov="1.3962634" />
+  </xacro:if>
 </robot>
