Commit message: Fixed gazebo stereo flag, added rules installation

File: wr8_description/urdf/model.urdf.xacro (robot description, xacro)
@@ -266,158 +266,158 @@
     </sensor>
   </gazebo>
+  <!-- Camera link -->
+  <xacro:macro name="camera_link" params="name">
+    <link name="${name}_frame">
+      <xacro:solid_cylinder_inertial
+          r="${camera_radius}" h="${camera_height}"
+          mass="${camera_mass}" >
+        <origin xyz="0 0 0" rpy="0 ${degrees_90} 0" />
+      </xacro:solid_cylinder_inertial>
+      <collision>
+        <origin xyz="0 0 0" rpy="0 ${degrees_90} 0" />
+        <geometry>
+          <cylinder length="${camera_height}" radius="${camera_radius}"/>
+        </geometry>
+      </collision>
+      <visual>
+        <origin xyz="0 0 0" rpy="0 ${degrees_90} 0" />
+        <geometry>
+          <cylinder length="${camera_height}" radius="${camera_radius}"/>
+        </geometry>
+      </visual>
+    </link>
+  </xacro:macro>
+  <!-- Single camera macro -->
+  <xacro:macro name="single_camera" params="name xyz rpy fov">
+    <xacro:camera_link name="${name}" />
+    <joint name="${name}_joint" type="fixed">
+      <child link="${name}_frame" />
+      <parent link="base_center" />
+      <origin xyz="${xyz}" rpy="${rpy}" />
+    </joint>
+    <link name="${name}_optical_frame"/>
+    <joint name="${name}_optical_frame_joint" type="fixed">
+      <origin xyz="0 0 0" rpy="-${degrees_90} 0.0 -${degrees_90}" />
+      <parent link="${name}_frame" />
+      <child link="${name}_optical_frame"/>
+    </joint>
+    <gazebo reference="${name}_frame">
+      <material>Gazebo/Black</material>
+      <sensor type="camera" name="${name}">
+        <update_rate>30.0</update_rate>
+        <camera name="${name}">
+          <horizontal_fov>${fov}</horizontal_fov>
+          <image>
+            <width>800</width>
+            <height>600</height>
+            <format>R8G8B8</format>
+          </image>
+          <clip>
+            <near>0.02</near>
+            <far>300</far>
+          </clip>
+          <noise>
+            <type>gaussian</type>
+            <mean>0.0</mean>
+            <stddev>0.001</stddev>
+          </noise>
+        </camera>
+        <plugin name="${name}_controller" filename="libgazebo_ros_camera.so">
+          <alwaysOn>true</alwaysOn>
+          <updateRate>30.0</updateRate>
+          <cameraName>$(arg robot_name)/${name}</cameraName>
+          <imageTopicName>image_raw</imageTopicName>
+          <cameraInfoTopicName>camera_info</cameraInfoTopicName>
+          <frameName>${name}_optical_frame</frameName>
+          <hackBaseline>0.07</hackBaseline>
+          <distortionK1>0.0</distortionK1>
+          <distortionK2>0.0</distortionK2>
+          <distortionK3>0.0</distortionK3>
+          <distortionT1>0.0</distortionT1>
+          <distortionT2>0.0</distortionT2>
+        </plugin>
+      </sensor>
+    </gazebo>
+  </xacro:macro>
+  <!-- Stereo camera macro -->
+  <xacro:macro name="stereo_camera" params="name fov">
+    <xacro:camera_link name="${name}_left" />
+    <xacro:camera_link name="${name}_right" />
+    <joint name="${name}_left_joint" type="fixed">
+      <child link="${name}_left_frame" />
+      <parent link="base_center" />
+      <origin xyz="${stereo_base_link_lcam_xyz}" rpy="0 0 0" />
+    </joint>
+    <joint name="${name}_right_joint" type="fixed">
+      <child link="${name}_right_frame" />
+      <parent link="base_center" />
+      <origin xyz="${stereo_base_link_rcam_xyz}" rpy="0 0 0" />
+    </joint>
+    <link name="${name}_optical_frame"/>
+    <joint name="${name}_optical_frame_joint" type="fixed">
+      <origin xyz="0 0 0" rpy="-${degrees_90} 0.0 -${degrees_90}" />
+      <parent link="${name}_left_frame" />
+      <child link="${name}_optical_frame"/>
+    </joint>
+    <gazebo reference="${name}_left_frame">
+      <material>Gazebo/Black</material>
+      <sensor type="multicamera" name="${name}">
+        <update_rate>30.0</update_rate>
+        <camera name="left">
+          <horizontal_fov>${fov}</horizontal_fov>
+          <image>
+            <width>800</width>
+            <height>600</height>
+            <format>R8G8B8</format>
+          </image>
+          <clip>
+            <near>0.02</near>
+            <far>300</far>
+          </clip>
+          <noise>
+            <type>gaussian</type>
+            <mean>0.0</mean>
+            <stddev>0.007</stddev>
+          </noise>
+        </camera>
+        <camera name="right">
+          <pose>0 -0.07 0 0 0 0</pose>
+          <!-- <pose>0 -0.035 0 0 0 0</pose> -->
+          <horizontal_fov>${fov}</horizontal_fov>
+          <image>
+            <width>800</width>
+            <height>600</height>
+            <format>R8G8B8</format>
+          </image>
+          <clip>
+            <near>0.02</near>
+            <far>300</far>
+          </clip>
+          <noise>
+            <type>gaussian</type>
+            <mean>0.0</mean>
+            <stddev>0.007</stddev>
+          </noise>
+        </camera>
+        <plugin name="${name}_controller" filename="libgazebo_ros_multicamera.so">
+          <alwaysOn>true</alwaysOn>
+          <updateRate>30.0</updateRate>
+          <cameraName>$(arg robot_name)/${name}</cameraName>
+          <imageTopicName>image_raw</imageTopicName>
+          <cameraInfoTopicName>camera_info</cameraInfoTopicName>
+          <frameName>${name}_optical_frame</frameName>
+          <hackBaseline>0.07</hackBaseline>
+          <distortionK1>0.0</distortionK1>
+          <distortionK2>0.0</distortionK2>
+          <distortionK3>0.0</distortionK3>
+          <distortionT1>0.0</distortionT1>
+          <distortionT2>0.0</distortionT2>
+        </plugin>
+      </sensor>
+    </gazebo>
+  </xacro:macro>
   <xacro:if value="$(arg enable_stereo)">
-    <!-- Camera link -->
-    <xacro:macro name="camera_link" params="name">
-      <link name="${name}_frame">
-        <xacro:solid_cylinder_inertial
-            r="${camera_radius}" h="${camera_height}"
-            mass="${camera_mass}" >
-          <origin xyz="0 0 0" rpy="0 ${degrees_90} 0" />
-        </xacro:solid_cylinder_inertial>
-        <collision>
-          <origin xyz="0 0 0" rpy="0 ${degrees_90} 0" />
-          <geometry>
-            <cylinder length="${camera_height}" radius="${camera_radius}"/>
-          </geometry>
-        </collision>
-        <visual>
-          <origin xyz="0 0 0" rpy="0 ${degrees_90} 0" />
-          <geometry>
-            <cylinder length="${camera_height}" radius="${camera_radius}"/>
-          </geometry>
-        </visual>
-      </link>
-    </xacro:macro>
-    <!-- Single camera macro -->
-    <xacro:macro name="single_camera" params="name xyz rpy fov">
-      <xacro:camera_link name="${name}" />
-      <joint name="${name}_joint" type="fixed">
-        <child link="${name}_frame" />
-        <parent link="base_center" />
-        <origin xyz="${xyz}" rpy="${rpy}" />
-      </joint>
-      <link name="${name}_optical_frame"/>
-      <joint name="${name}_optical_frame_joint" type="fixed">
-        <origin xyz="0 0 0" rpy="-${degrees_90} 0.0 -${degrees_90}" />
-        <parent link="${name}_frame" />
-        <child link="${name}_optical_frame"/>
-      </joint>
-      <gazebo reference="${name}_frame">
-        <material>Gazebo/Black</material>
-        <sensor type="camera" name="${name}">
-          <update_rate>30.0</update_rate>
-          <camera name="${name}">
-            <horizontal_fov>${fov}</horizontal_fov>
-            <image>
-              <width>800</width>
-              <height>600</height>
-              <format>R8G8B8</format>
-            </image>
-            <clip>
-              <near>0.02</near>
-              <far>300</far>
-            </clip>
-            <noise>
-              <type>gaussian</type>
-              <mean>0.0</mean>
-              <stddev>0.001</stddev>
-            </noise>
-          </camera>
-          <plugin name="${name}_controller" filename="libgazebo_ros_camera.so">
-            <alwaysOn>true</alwaysOn>
-            <updateRate>30.0</updateRate>
-            <cameraName>$(arg robot_name)/${name}</cameraName>
-            <imageTopicName>image_raw</imageTopicName>
-            <cameraInfoTopicName>camera_info</cameraInfoTopicName>
-            <frameName>${name}_optical_frame</frameName>
-            <hackBaseline>0.07</hackBaseline>
-            <distortionK1>0.0</distortionK1>
-            <distortionK2>0.0</distortionK2>
-            <distortionK3>0.0</distortionK3>
-            <distortionT1>0.0</distortionT1>
-            <distortionT2>0.0</distortionT2>
-          </plugin>
-        </sensor>
-      </gazebo>
-    </xacro:macro>
-    <!-- Stereo camera macro -->
-    <xacro:macro name="stereo_camera" params="name fov">
-      <xacro:camera_link name="${name}_left" />
-      <xacro:camera_link name="${name}_right" />
-      <joint name="${name}_left_joint" type="fixed">
-        <child link="${name}_left_frame" />
-        <parent link="base_center" />
-        <origin xyz="${stereo_base_link_lcam_xyz}" rpy="0 0 0" />
-      </joint>
-      <joint name="${name}_right_joint" type="fixed">
-        <child link="${name}_right_frame" />
-        <parent link="base_center" />
-        <origin xyz="${stereo_base_link_rcam_xyz}" rpy="0 0 0" />
-      </joint>
-      <link name="${name}_optical_frame"/>
-      <joint name="${name}_optical_frame_joint" type="fixed">
-        <origin xyz="0 0 0" rpy="-${degrees_90} 0.0 -${degrees_90}" />
-        <parent link="${name}_left_frame" />
-        <child link="${name}_optical_frame"/>
-      </joint>
-      <gazebo reference="${name}_left_frame">
-        <material>Gazebo/Black</material>
-        <sensor type="multicamera" name="${name}">
-          <update_rate>30.0</update_rate>
-          <camera name="left">
-            <horizontal_fov>${fov}</horizontal_fov>
-            <image>
-              <width>800</width>
-              <height>600</height>
-              <format>R8G8B8</format>
-            </image>
-            <clip>
-              <near>0.02</near>
-              <far>300</far>
-            </clip>
-            <noise>
-              <type>gaussian</type>
-              <mean>0.0</mean>
-              <stddev>0.007</stddev>
-            </noise>
-          </camera>
-          <camera name="right">
-            <pose>0 -0.07 0 0 0 0</pose>
-            <!-- <pose>0 -0.035 0 0 0 0</pose> -->
-            <horizontal_fov>${fov}</horizontal_fov>
-            <image>
-              <width>800</width>
-              <height>600</height>
-              <format>R8G8B8</format>
-            </image>
-            <clip>
-              <near>0.02</near>
-              <far>300</far>
-            </clip>
-            <noise>
-              <type>gaussian</type>
-              <mean>0.0</mean>
-              <stddev>0.007</stddev>
-            </noise>
-          </camera>
-          <plugin name="${name}_controller" filename="libgazebo_ros_multicamera.so">
-            <alwaysOn>true</alwaysOn>
-            <updateRate>30.0</updateRate>
-            <cameraName>$(arg robot_name)/${name}</cameraName>
-            <imageTopicName>image_raw</imageTopicName>
-            <cameraInfoTopicName>camera_info</cameraInfoTopicName>
-            <frameName>${name}_optical_frame</frameName>
-            <hackBaseline>0.07</hackBaseline>
-            <distortionK1>0.0</distortionK1>
-            <distortionK2>0.0</distortionK2>
-            <distortionK3>0.0</distortionK3>
-            <distortionT1>0.0</distortionT1>
-            <distortionT2>0.0</distortionT2>
-          </plugin>
-        </sensor>
-      </gazebo>
-    </xacro:macro>
     <xacro:stereo_camera name="stereo_camera" fov="1.3962634" />
-    <xacro:single_camera name="signs_camera" xyz="-0.05 0 0.3" rpy="0 -${degrees_30} -${degrees_30}" fov="1.3962634" />
   </xacro:if>
+  <xacro:single_camera name="signs_camera" xyz="-0.05 0 0.3" rpy="0 -${degrees_30} -${degrees_30}" fov="1.3962634" />
 </robot>
